File: AESIR_PCB_MB/AESIR_PCB_MB.sch (KiCad schematic (older format))
At the start: 33 parts, among them J1 Umb - GND, J10 GPS - Rx, J12 Saftey Pin - 5V - IN, J13 Saftey Pin - 5V - OUT, J14 Saftey Pin - 5V, J15 Vin - +5.5V, J16 Servo - 5V, J17 Servo - GND, J18 GPS - Tx, J19 Tel - GND, J2 Go Pro - 5V, J20 Tel - Rx, J21 Tel - Tx, J3 Umb - Rx, J4 Umb - Tx, J5 Umb - 5V, J6 Go Pro - GND, J8 GPS - GND, J9 M3 Drain - Tx Video/Cam, Q1 Q_NMOS_DGS, Q2 Q_NMOS_DGS, Q3 Q_NMOS_DGS, U1 Teensy3.6, U2 MPU-9250, U3 BMP180, U4 AESIR_MOTHERBOARD_PLATE

Commit message: finalized motherboard design, added library files
Parts:
- U4: footprint Enclosures:AESIR_MB_OUTLINE_68mm -> AESIR:AESIR_MB_OUTLINE_68mm
Changed lines of the file:
@@
 LIBS:contrib
 LIBS:valves
-LIBS:AESIR
 LIBS:teensy
 LIBS:AESIR_PCB_MB-cache
@@
 F 0 "U4" H 9200 3700 60  0000 C CNN
 F 1 "AESIR_MOTHERBOARD_PLATE" H 6850 7000 60  0000 C CNN
-F 2 "Enclosures:AESIR_MB_OUTLINE_68mm" H 6900 3650 60  0001 C CNN
+F 2 "AESIR:AESIR_MB_OUTLINE_68mm" H 6900 3650 60  0001 C CNN
 F 3 "" H 6900 3650 60  0001 C CNN
 	1    6850 3650
